Commit message: Trying to attach gripper on UR10

File: src/painting_robot/urdf/painting_robot.urdf.xacro (robot description, xacro)
@@ -31,3 +31,8 @@
     <origin xyz="0.0 0.0 0.0" rpy="0.0 0.0 0.0" />
   </joint>
+  <joint name="UR10_and_gripper_joint" type="fixed">
+    <parent link="arm_ee_link" />
+    <child link = "palm" />
+    <origin xyz="0.0 0.0 0.0" rpy="0.0 0.0 0.0" />
+  </joint>
 </robot>

Commit message: Commented gripper model as it was causing errors

File: src/painting_robot/urdf/painting_robot.urdf.xacro (robot description, xacro)
@@ -31,8 +31,8 @@
     <origin xyz="0.0 0.0 0.0" rpy="0.0 0.0 0.0" />
   </joint>
-  <joint name="UR10_and_gripper_joint" type="fixed">
+  <!--joint name="UR10_and_gripper_joint" type="fixed">
     <parent link="arm_ee_link" />
     <child link = "palm" />
     <origin xyz="0.0 0.0 0.0" rpy="0.0 0.0 0.0" />
-  </joint>
+  </joint-->
 </robot>
